Commit message: descriptions added

File: catkin_ws/src/robot_modelling/urdf/instructional_robot_body.xacro (robot description, xacro)
@@ -10,6 +10,6 @@
   <xacro:instructional_robot_wheels xyz_position="0.0 -0.175 -0.1" rpy_position="0 0 0" direction="left"/>
   <xacro:instructional_robot_wheels xyz_position="0.0 0.175 -0.1" rpy_position="0 0 0" direction="right"/>
-  <xacro:instructional_robot_castor_wheels xyz_position="0.2 0.0 -0.15" rpy_position="0 0 0" direction="front"/>
-  <xacro:instructional_robot_castor_wheels xyz_position="-0.2 0.0 -0.15" rpy_position="0 0 0" direction="back"/>
+  <xacro:instructional_robot_caster_wheels xyz_position="0.2 0.0 -0.15" rpy_position="0 0 0" direction="front"/>
+  <xacro:instructional_robot_caster_wheels xyz_position="-0.2 0.0 -0.15" rpy_position="0 0 0" direction="back"/>
   <xacro:instructional_robot_differential />
   <xacro:instructional_robot_laser />

File: catkin_ws/src/robot_modelling/urdf/instructional_robot_wheels.xacro (robot description, xacro)
@@ -27,5 +27,5 @@
   </gazebo>
   </xacro:macro>
-  <xacro:macro name="instructional_robot_castor_wheels" params="xyz_position rpy_position direction">
+  <xacro:macro name="instructional_robot_caster_wheels" params="xyz_position rpy_position direction">
   <link name="caster_wheel_${direction}_link">
     <collision>
